File: PCB/main/main.kicad_sch (KiCad schematic)
At the start: 4 parts, among them J1 Conn_01x33_Female, J2 Conn_01x33_Female, J3 Conn_01x33_Female, J4 Conn_01x33_Female

Commit message: v1.0 BOM, Gerbers & Final Designs
Parts:
- added D1: Red LED, Red_LED:LEDC1608X70N, symbol Device:LED
Connections:
- net GND: now also D1.1 (K)
- net Power/USBDETECT: now also D1.2 (A)
- no-connect marks 2 -> 0
Other:
- sheet microcontroller_interfacing ports: added USB(+5); removed none
