File: PCB/main/microcontroller_interfacing.kicad_sch (KiCad schematic)
At the start: 0 parts

Commit message: Added sheet details to schematic
Other:
- company: (none) -> UCT
Changed lines of the file:
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@@
 (kicad_sch (version 20211123) (generator eeschema)
   (paper "A4")
+  (title_block
+    (date "2022-03-02")
+    (rev "v0.0")
+    (company "UCT")
+    (comment 2 "Group 7")
+    (comment 3 "@Checked By: ")
+    (comment 4 "@Authors: Ryan Jones, Alex Cargill & Devlin Trafford")
+  )
   (text "Memory Element and which pins you wish to use.\ndebugging capabilities to test it\n"
     (at 129.54 89.535 0)

Commit message: uC SubModule v0.01
Parts:
- added C6: 0.1u, symbol pspice:CAP
- added C7: 47nF, symbol pspice:CAP
- added C8, C9: 22p, symbol pspice:CAP
- added IC3: M24C02-WMN6TP, symbol M24C02-WMN6TP:M24C02-WMN6TP
- added J6, J7, J8: Conn_01x01_Female, symbol Connector:Conn_01x01_Female
- added R17, R18: 4.7k, symbol Device:R_US
- added U2: CH340G, Package_SO:SOIC-16_3.9x9.9mm_P1.27mm, symbol Interface_USB:CH340G
- added Y1: Crystal, symbol Device:Crystal
Connections:
- new net: C8.1, U2.7 (XI), Y1.1
- new net: C9.1, U2.8 (XO), Y1.2
- new net GND: C6.2, C7.2, C8.2, C9.2, IC3.2 (E1), IC3.3 (E2), IC3.4 (VSS), U2.1 (GND)
- new net PA0: IC3.7 (~{WC})
- new net PA1: J6.1 (Pin_1)
- new net PA2: J7.1 (Pin_1)
- new net PA3: J8.1 (Pin_1)
- new net PB6: U2.3 (RXD)
- new net PB7: U2.2 (TXD)
- new net PB8: IC3.5 (SDA), R17.2
- new net PB9: IC3.6 (SCL), R18.2
- new net PC1: U2.9 (~{CTS})
- new net PC2: U2.10 (~{DSR})
- new net PC3: U2.11 (~{RI})
- new net PC4: U2.12 (~{DCD}), U2.13 (~{DTR})
- new net PC5: U2.14 (~{RTS})
- new net PWR (3.3V): C6.1, C7.1, IC3.1 (E0), IC3.8 (VCC), R17.1, R18.1, U2.16 (VCC), U2.4 (V3)
- new net USB (D+): U2.5 (UD+)
- new net USB (D-): U2.6 (UD-)
Other:
- note removed: "Memory Element and which pins you wish to use. debugging capabilities to test it"
- title: (none) -> Microcontroller Interfacing

Commit message: Power v0.1, Sensing v0.1, uC Control v0.1, Simulations
Parts:
- R16: renamed from R17; JLC Part Number (none) -> C17673; Price (none) -> 0.0027
- R17: renamed from R18; JLC Part Number (none) -> C17673; Price (none) -> 0.0027
- renumbered C8 to C10, C9 to C11, C7 to C8, C6 to C9, U2 to U4
Connections:
- net PA1 renamed S1 (Digital Sensor)
- net PA2 renamed S2 (Analog Sensor)
- net PA3 renamed S3 (Analog Sensor)
Changed lines of the file:
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@@
   (title_block
     (title "Microcontroller Interfacing")
-    (date "2022-03-04")
-    (rev "v0.0")
+    (date "2022-03-11")
+    (rev "v0.10")
     (company "UCT")
     (comment 2 "Group 7")
@@
     (stroke (width 0) (type default) (color 0 0 0 0))
   )
+  (label "PC2" (at 110.49 147.32 0)
+    (effects (font (size 1.27 1.27)) (justify left bottom))
+  )
+  (label "PA0" (at 125.73 54.61 0)
+    (effects (font (size 1.27 1.27)) (justify left bottom))
+  )
+  (label "PC1" (at 110.49 144.78 0)
+    (effects (font (size 1.27 1.27)) (justify left bottom))
+  )
+  (label "PA2" (at 157.48 110.49 0)
+    (effects (font (size 1.27 1.27)) (justify left bottom))
+  )
+  (label "PA3" (at 158.75 149.86 0)
+    (effects (font (size 1.27 1.27)) (justify left bottom))
+  )
+  (label "PB8" (at 125.73 59.69 0)
+    (effects (font (size 1.27 1.27)) (justify left bottom))
+  )
+  (label "PA1" (at 157.48 68.58 0)
+    (effects (font (size 1.27 1.27)) (justify left bottom))
+  )
+  (label "PB7" (at 110.49 137.16 0)
+    (effects (font (size 1.27 1.27)) (justify left bottom))
+  )
+  (label "PC5" (at 110.49 157.48 0)
+    (effects (font (size 1.27 1.27)) (justify left bottom))
+  )
+  (label "PB6" (at 110.49 139.7 0)
+    (effects (font (size 1.27 1.27)) (justify left bottom))
+  )
+  (label "PC4" (at 110.49 154.94 0)
+    (effects (font (size 1.27 1.27)) (justify left bottom))
+  )
+  (label "PC3" (at 110.49 149.86 0)
+    (effects (font (size 1.27 1.27)) (justify left bottom))
+  )
+  (label "PB9" (at 125.73 57.15 0)
+    (effects (font (size 1.27 1.27)) (justify left bottom))
+  )
+  (label "PC4" (at 110.49 152.4 0)
+    (effects (font (size 1.27 1.27)) (justify left bottom))
+  )
   (hierarchical_label "USB (D-)" (shape input) (at 50.8 114.3 180)
     (effects (font (size 1.27 1.27)) (justify right))
   )
-  (hierarchical_label "PC1" (shape input) (at 110.49 144.78 0)
-    (effects (font (size 1.27 1.27)) (justify left))
-  )
-  (hierarchical_label "PA3" (shape input) (at 158.75 149.86 0)
-    (effects (font (size 1.27 1.27)) (justify left))
-  )
-  (hierarchical_label "PC4" (shape input) (at 110.49 152.4 0)
-    (effects (font (size 1.27 1.27)) (justify left))
-  )
-  (hierarchical_label "PA0" (shape input) (at 125.73 54.61 0)
-    (effects (font (size 1.27 1.27)) (justify left))
-  )
   (hierarchical_label "PWR (3.3V)" (shape input) (at 80.01 24.13 0)
     (effects (font (size 1.27 1.27)) (justify left))
   )
-  (hierarchical_label "PB7" (shape input) (at 110.49 137.16 0)
-    (effects (font (size 1.27 1.27)) (justify left))
-  )
-  (hierarchical_label "PA1" (shape input) (at 157.48 68.58 0)
-    (effects (font (size 1.27 1.27)) (justify left))
-  )
-  (hierarchical_label "PC4" (shape input) (at 110.49 154.94 0)
-    (effects (font (size 1.27 1.27)) (justify left))
-  )
   (hierarchical_label "USB (D+)" (shape input) (at 54.61 114.3 0)
     (effects (font (size 1.27 1.27)) (justify left))
@@
     (effects (font (size 1.27 1.27)) (justify left))
   )
-  (hierarchical_label "PC5" (shape input) (at 110.49 157.48 0)
-    (effects (font (size 1.27 1.27)) (justify left))
-  )
   (hierarchical_label "S1 (Digital Sensor)" (shape input) (at 157.48 40.64 0)
     (effects (font (size 1.27 1.27)) (justify left))
   )
-  (hierarchical_label "PB6" (shape input) (at 110.49 139.7 0)
-    (effects (font (size 1.27 1.27)) (justify left))
-  )
-  (hierarchical_label "PC3" (shape input) (at 110.49 149.86 0)
-    (effects (font (size 1.27 1.27)) (justify left))
-  )
   (hierarchical_label "S2 (Analog Sensor)" (shape input) (at 157.48 82.55 0)
     (effects (font (size 1.27 1.27)) (justify left))
   )
-  (hierarchical_label "PB8" (shape input) (at 125.73 59.69 0)
-    (effects (font (size 1.27 1.27)) (justify left))
-  )
   (hierarchical_label "PWR (3.3V)" (shape input) (at 26.67 29.21 0)
     (effects (font (size 1.27 1.27)) (justify left))
   )
-  (hierarchical_label "PB9" (shape input) (at 125.73 57.15 0)
-    (effects (font (size 1.27 1.27)) (justify left))
-  )
-  (hierarchical_label "PA2" (shape input) (at 157.48 110.49 0)
-    (effects (font (size 1.27 1.27)) (justify left))
-  )
   (hierarchical_label "PWR (3.3V)" (shape input) (at 25.4 118.11 0)
     (effects (font (size 1.27 1.27)) (justify left))
   )
-  (hierarchical_label "PC2" (shape input) (at 110.49 147.32 0)
-    (effects (font (size 1.27 1.27)) (justify left))
-  )
   (symbol (lib_id "pspice:CAP") (at 33.02 171.45 0) (unit 1)
     (in_bom yes) (on_board yes) (fields_autoplaced)
-    (property "Reference" "C8" (id 0) (at 38.1 170.1799 0)
+    (property "Reference" "C10" (id 0) (at 38.1 170.1799 0)
       (effects (font (size 1.27 1.27)) (justify left))
     )
@@
   (symbol (lib_id "power:GND") (at 26.67 59.69 0) (unit 1)
     (in_bom yes) (on_board yes) (fields_autoplaced)
-    (property "Reference" "#PWR020" (id 0) (at 26.67 66.04 0)
+    (property "Reference" "#PWR038" (id 0) (at 26.67 66.04 0)
       (effects (font (size 1.27 1.27)) hide)
     )
@@
   (symbol (lib_id "pspice:CAP") (at 54.61 172.72 0) (unit 1)
     (in_bom yes) (on_board yes) (fields_autoplaced)
-    (property "Reference" "C9" (id 0) (at 59.69 171.4499 0)
+    (property "Reference" "C11" (id 0) (at 59.69 171.4499 0)
       (effects (font (size 1.27 1.27)) (justify left))
     )
@@
   (symbol (lib_id "Interface_USB:CH340G") (at 71.12 147.32 0) (unit 1)
     (in_bom yes) (on_board yes) (fields_autoplaced)
-    (property "Reference" "U2" (id 0) (at 73.1394 162.56 0)
+    (property "Reference" "U4" (id 0) (at 73.1394 162.56 0)
       (effects (font (size 1.27 1.27)) (justify left))
     )
@@
   (symbol (lib_id "power:GND") (at 25.4 180.34 0) (unit 1)
     (in_bom yes) (on_board yes) (fields_autoplaced)
-    (property "Reference" "#PWR019" (id 0) (at 25.4 186.69 0)
+    (property "Reference" "#PWR040" (id 0) (at 25.4 186.69 0)
       (effects (font (size 1.27 1.27)) hide)
     )
@@
   (symbol (lib_id "pspice:CAP") (at 26.67 49.53 0) (unit 1)
     (in_bom yes) (on_board yes) (fields_autoplaced)
-    (property "Reference" "C7" (id 0) (at 31.75 48.2599 0)
+    (property "Reference" "C8" (id 0) (at 31.75 48.2599 0)
       (effects (font (size 1.27 1.27)) (justify left))
     )
@@
   (symbol (lib_id "pspice:CAP") (at 25.4 142.24 0) (unit 1)
     (in_bom yes) (on_board yes) (fields_autoplaced)
-    (property "Reference" "C6" (id 0) (at 30.48 140.9699 0)
+    (property "Reference" "C9" (id 0) (at 30.48 140.9699 0)
       (effects (font (size 1.27 1.27)) (justify left))
     )
@@
   (symbol (lib_id "power:GND") (at 48.26 85.09 0) (unit 1)
     (in_bom yes) (on_board yes) (fields_autoplaced)
-    (property "Reference" "#PWR021" (id 0) (at 48.26 91.44 0)
+    (property "Reference" "#PWR039" (id 0) (at 48.26 91.44 0)
       (effects (font (size 1.27 1.27)) hide)
     )
@@
   (symbol (lib_id "Device:R_US") (at 111.76 44.45 0) (unit 1)
     (in_bom yes) (on_board yes) (fields_autoplaced)
-    (property "Reference" "R18" (id 0) (at 114.3 43.1799 0)
+    (property "Reference" "R17" (id 0) (at 114.3 43.1799 0)
       (effects (font (size 1.27 1.27)) (justify left))
     )
@@
       (effects (font (size 1.27 1.27)) hide)
     )
+    (property "JLC Part Number" "C17673" (id 4) (at 111.76 44.45 0)
+      (effects (font (size 1.27 1.27)) hide)
+    )
+    (property "Price" "0.0027" (id 5) (at 111.76 44.45 0)
+      (effects (font (size 1.27 1.27)) hide)
+    )
     (pin "1")
     (pin "2")
@@
   (symbol (lib_id "Device:R_US") (at 87.63 44.45 0) (unit 1)
     (in_bom yes) (on_board yes) (fields_autoplaced)
-    (property "Reference" "R17" (id 0) (at 90.17 43.1799 0)
+    (property "Reference" "R16" (id 0) (at 90.17 43.1799 0)
       (effects (font (size 1.27 1.27)) (justify left))
     )
@@
       (effects (font (size 1.27 1.27)) hide)
     )
+    (property "JLC Part Number" "C17673" (id 4) (at 87.63 44.45 0)
+      (effects (font (size 1.27 1.27)) hide)
+    )
+    (property "Price" "0.0027" (id 5) (at 87.63 44.45 0)
+      (effects (font (size 1.27 1.27)) hide)
+    )
