File: PCB/main/microcontroller_interfacing.kicad_sch (KiCad schematic)
At the start: 12 parts, among them IC3 M24C02-WMN6TP, J10 Conn_01x01_Female, J11 Conn_01x01_Female, J12 Conn_01x01_Female, U4 CH340G, Y1 Crystal

Commit message: Power, uC, Sensing v0.1.1
Parts:
- removed C10: 0.1u, symbol pspice:CAP
- removed C11, C12: 22p, symbol pspice:CAP
- removed C9: 47nF, symbol pspice:CAP
- removed IC3: M24C02-WMN6TP, symbol M24C02-WMN6TP:M24C02-WMN6TP
- removed J10, J11, J12: Conn_01x01_Female, symbol Connector:Conn_01x01_Female
- removed R14, R15: 4.7k, symbol Device:R_US
- removed Y1: Crystal, symbol Device:Crystal
- added C10, C11: 100n, Capacitor_SMD:C_0402_1005Metric, symbol CL05B104KO5NNNC:CL05B104KO5NNNC
- added C12, C13: 22p, Capacitor_SMD:C_0805_2012Metric, symbol CL05B104KO5NNNC:CL05B104KO5NNNC
- added C9: 47n, Capacitor_SMD:C_0603_1608Metric, symbol CL05B104KO5NNNC:CL05B104KO5NNNC
- added D6, D7, D8: LED, LED_SMD:LED_0805_2012Metric, symbol Device:LED
- added IC3: AT24C256C-SSHL-T, EEPROM:SOIC127P600X175-8N, symbol AT24C256C-SSHL-T:AT24C256C-SSHL-T
- added R18, R19: 4.7k, Resistor_SMD:R_0402_1005Metric, symbol 0402WGF4701TCE:0402WGF4701TCE
- added R20, R21, R22: 1.5k, Resistor_SMD:R_0402_1005Metric, symbol 0402WGF4701TCE:0402WGF4701TCE
- added TP10, TP11, TP12, TP8, TP9: TestPoint, TestPoint:TestPoint_Pad_D2.5mm, symbol Connector:TestPoint
- added Y1: YSX321SL, YSX321SL:YSX321SL, symbol YSX321SL:YSX321SL
- U4: footprint Package_SO:SOIC-16_3.9x9.9mm_P1.27mm -> CH340G:SOIC127P600X180-16N
Connections:
- net GND: now also C10.1, C11.1, C12.1, C13.1, C9.1, IC3.1 (A0), IC3.2 (A1), IC3.3 (A2), IC3.4 (GND), R22.1
- net PB6: now also IC3.6 (SCL), R19.1, TP9.1; no longer U4.3 (RXD)
- net PB7: now also IC3.5 (SDA), R18.1, TP10.1; no longer U4.2 (TXD)
- net at U4.7 (XI): now also Y1.1 (CRYSTAL_1)
- net at U4.8 (XO): now also Y1.3 (CRYSTAL_2)
- net PC1: no longer names the net of U4.9 (~{CTS})
- net PC2: no longer names the net of U4.10 (~{DSR})
- net PC3: no longer names the net of U4.11 (~{RI})
- net PC4: no longer names the net of U4.12 (~{DCD})
- net PC4: no longer U4.13 (~{DTR})
- net PC5: no longer names the net of U4.14 (~{RTS})
- net PWR (3.3V) renamed 3V3
- net 3V3: now also C10.2, C11.2, C9.2, D6.2 (A), D7.2 (A), D8.2 (A), IC3.8 (VCC), R18.2, R19.2
- new net: D6.1 (K), R20.2
- new net: C13.2, Y1.2 (GND_1)
- new net: C12.2, Y1.4 (GND_2)
- new net: D7.1 (K), R21.2
- new net PA10: R21.1, TP12.1, U4.2 (TXD)
- new net PA3: IC3.7 (WP), TP8.1
- new net PA9: D8.1 (K), R20.1, R22.2, TP11.1, U4.3 (RXD)
- no-connect marks 1 -> 7
Other:
- note added: "v0.1: -Changed EEPROM to AT24C256C-SSHL-T -Changed Power Connections for CH340G -Added LEDs in order to see if power is flowing in traces."

Commit message: Schematics v0.1.1 & PCB v0.01
Parts:
- C12, C13: footprint Capacitor_SMD:C_0805_2012Metric -> 22pF_0804:CAPC1608X90N
- C9: footprint Capacitor_SMD:C_0603_1608Metric -> 47nF_0804:CAPC1608X90N
- IC3: footprint EEPROM:SOIC127P600X175-8N -> 3088_uC:SOIC127P600X175-8N
- R18, R19, R20, R21, R22: footprint Resistor_SMD:R_0402_1005Metric -> 4k7:RESC2013X65N
- TP10: renamed from TP9; footprint TestPoint:TestPoint_Pad_D2.5mm -> TestPoint:TestPoint_Pad_D2.0mm
- TP11: renamed from TP10; footprint TestPoint:TestPoint_Pad_D2.5mm -> TestPoint:TestPoint_Pad_D2.0mm
- TP12: renamed from TP11; footprint TestPoint:TestPoint_Pad_D2.5mm -> TestPoint:TestPoint_Pad_D2.0mm
- TP13: renamed from TP12; footprint TestPoint:TestPoint_Pad_D2.5mm -> TestPoint:TestPoint_Pad_D2.0mm
- TP9: renamed from TP8; footprint TestPoint:TestPoint_Pad_D2.5mm -> TestPoint:TestPoint_Pad_D2.0mm
- U4: footprint CH340G:SOIC127P600X180-16N -> 3088_uC:SOIC127P600X180-16N
- Y1: footprint YSX321SL:YSX321SL -> 3088_uC:YSX321SL
Changed lines of the file:
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@@
       (effects (font (size 1.27 1.27)) (justify right))
     )
-    (property "Footprint" "Resistor_SMD:R_0402_1005Metric" (id 2) (at 156.21 85.09 0)
+    (property "Footprint" "4k7:RESC2013X65N" (id 2) (at 156.21 85.09 0)
       (effects (font (size 1.27 1.27)) (justify left) hide)
     )
@@
       (effects (font (size 1.27 1.27)) (justify left))
     )
-    (property "Footprint" "CH340G:SOIC127P600X180-16N" (id 2) (at 73.66 113.03 0)
+    (property "Footprint" "3088_uC:SOIC127P600X180-16N" (id 2) (at 73.66 113.03 0)
       (effects (font (size 1.27 1.27)) (justify left) hide)
     )
@@
       (effects (font (size 1.27 1.27)) (justify right))
     )
-    (property "Footprint" "Capacitor_SMD:C_0603_1608Metric" (id 2) (at 15.24 36.83 0)
+    (property "Footprint" "47nF_0804:CAPC1608X90N" (id 2) (at 15.24 36.83 0)
       (effects (font (size 1.27 1.27)) (justify left) hide)
     )
@@
     (property "Reference" "Y1" (id 0) (at 39.37 102.87 0))
     (property "Value" "YSX321SL" (id 1) (at 39.37 105.41 0))
-    (property "Footprint" "YSX321SL:YSX321SL" (id 2) (at 55.88 107.95 0)
+    (property "Footprint" "3088_uC:YSX321SL" (id 2) (at 55.88 107.95 0)
       (effects (font (size 1.27 1.27)) (justify left) hide)
     )
@@
   (symbol (lib_id "power:GND") (at 16.51 49.53 0) (unit 1)
     (in_bom yes) (on_board yes) (fields_autoplaced)
-    (property "Reference" "#PWR042" (id 0) (at 16.51 55.88 0)
+    (property "Reference" "#PWR043" (id 0) (at 16.51 55.88 0)
       (effects (font (size 1.27 1.27)) hide)
     )
@@
   (symbol (lib_id "Connector:TestPoint") (at 146.05 97.155 0) (unit 1)
     (in_bom yes) (on_board yes) (fields_autoplaced)
-    (property "Reference" "TP12" (id 0) (at 148.59 92.5829 0)
+    (property "Reference" "TP13" (id 0) (at 148.59 92.5829 0)
       (effects (font (size 1.27 1.27)) (justify left))
     )
@@
       (effects (font (size 1.27 1.27)) (justify left))
     )
-    (property "Footprint" "TestPoint:TestPoint_Pad_D2.5mm" (id 2) (at 151.13 97.155 0)
+    (property "Footprint" "TestPoint:TestPoint_Pad_D2.0mm" (id 2) (at 151.13 97.155 0)
       (effects (font (size 1.27 1.27)) hide)
     )
@@
   (symbol (lib_id "power:GND") (at 48.26 91.44 180) (unit 1)
     (in_bom yes) (on_board yes) (fields_autoplaced)
-    (property "Reference" "#PWR044" (id 0) (at 48.26 85.09 0)
+    (property "Reference" "#PWR045" (id 0) (at 48.26 85.09 0)
       (effects (font (size 1.27 1.27)) hide)
     )
@@
   (symbol (lib_id "power:GND") (at 31.75 58.42 0) (unit 1)
     (in_bom yes) (on_board yes) (fields_autoplaced)
-    (property "Reference" "#PWR043" (id 0) (at 31.75 64.77 0)
+    (property "Reference" "#PWR044" (id 0) (at 31.75 64.77 0)
       (effects (font (size 1.27 1.27)) hide)
     )
@@
   (symbol (lib_id "Connector:TestPoint") (at 107.95 36.83 0) (unit 1)
     (in_bom yes) (on_board yes) (fields_autoplaced)
-    (property "Reference" "TP8" (id 0) (at 110.49 32.2579 0)
+    (property "Reference" "TP9" (id 0) (at 110.49 32.2579 0)
       (effects (font (size 1.27 1.27)) (justify left))
     )
@@
       (effects (font (size 1.27 1.27)) (justify left))
     )
-    (property "Footprint" "TestPoint:TestPoint_Pad_D2.5mm" (id 2) (at 113.03 36.83 0)
+    (property "Footprint" "TestPoint:TestPoint_Pad_D2.0mm" (id 2) (at 113.03 36.83 0)
       (effects (font (size 1.27 1.27)) hide)
     )
@@
     (property "Reference" "IC3" (id 0) (at 43.18 26.67 0))
     (property "Value" "AT24C256C-SSHL-T" (id 1) (at 43.18 29.21 0))
-    (property "Footprint" "EEPROM:SOIC127P600X175-8N" (id 2) (at 53.34 31.75 0)
+    (property "Footprint" "3088_uC:SOIC127P600X175-8N" (id 2) (at 53.34 31.75 0)
       (effects (font (size 1.27 1.27)) (justify left) hide)
     )
@@
   (symbol (lib_id "Connector:TestPoint") (at 64.77 41.91 0) (unit 1)
     (in_bom yes) (on_board yes) (fields_autoplaced)
-    (property "Reference" "TP10" (id 0) (at 67.31 37.3379 0)
+    (property "Reference" "TP11" (id 0) (at 67.31 37.3379 0)
       (effects (font (size 1.27 1.27)) (justify left))
     )
@@
       (effects (font (size 1.27 1.27)) (justify left))
     )
-    (property "Footprint" "TestPoint:TestPoint_Pad_D2.5mm" (id 2) (at 69.85 41.91 0)
+    (property "Footprint" "TestPoint:TestPoint_Pad_D2.0mm" (id 2) (at 69.85 41.91 0)
       (effects (font (size 1.27 1.27)) hide)
     )
@@
   (symbol (lib_id "power:GND") (at 86.36 133.35 0) (unit 1)
     (in_bom yes) (on_board yes) (fields_autoplaced)
-    (property "Reference" "#PWR046" (id 0) (at 86.36 139.7 0)
+    (property "Reference" "#PWR047" (id 0) (at 86.36 139.7 0)
       (effects (font (size 1.27 1.27)) hide)
     )
@@
       (effects (font (size 1.27 1.27)) (justify right))
     )
-    (property "Footprint" "Resistor_SMD:R_0402_1005Metric" (id 2) (at 73.66 21.59 0)
+    (property "Footprint" "4k7:RESC2013X65N" (id 2) (at 73.66 21.59 0)
       (effects (font (size 1.27 1.27)) (justify left) hide)
     )
@@
       (effects (font (size 1.27 1.27)) (justify right))
     )
-    (property "Footprint" "Capacitor_SMD:C_0805_2012Metric" (id 2) (at 20.32 121.92 0)
+    (property "Footprint" "22pF_0804:CAPC1608X90N" (id 2) (at 20.32 121.92 0)
       (effects (font (size 1.27 1.27)) (justify left) hide)
     )
@@
       (effects (font (size 1.27 1.27)) (justify right))
     )
-    (property "Footprint" "Capacitor_SMD:C_0805_2012Metric" (id 2) (at 41.91 123.19 0)
+    (property "Footprint" "22pF_0804:CAPC1608X90N" (id 2) (at 41.91 123.19 0)
       (effects (font (size 1.27 1.27)) (justify left) hide)
     )
@@
   (symbol (lib_id "Connector:TestPoint") (at 85.09 39.37 0) (unit 1)
     (in_bom yes) (on_board yes) (fields_autoplaced)
-    (property "Reference" "TP9" (id 0) (at 87.63 34.7979 0)
+    (property "Reference" "TP10" (id 0) (at 87.63 34.7979 0)
       (effects (font (size 1.27 1.27)) (justify left))
     )
@@
       (effects (font (size 1.27 1.27)) (justify left))
     )
-    (property "Footprint" "TestPoint:TestPoint_Pad_D2.5mm" (id 2) (at 90.17 39.37 0)
+    (property "Footprint" "TestPoint:TestPoint_Pad_D2.0mm" (id 2) (at 90.17 39.37 0)
       (effects (font (size 1.27 1.27)) hide)
     )
@@
       (effects (font (size 1.27 1.27)) (justify right))
     )
-    (property "Footprint" "Resistor_SMD:R_0402_1005Metric" (id 2) (at 93.98 21.59 0)
+    (property "Footprint" "4k7:RESC2013X65N" (id 2) (at 93.98 21.59 0)
       (effects (font (size 1.27 1.27)) (justify left) hide)
     )
@@
   (symbol (lib_id "power:GND") (at 125.73 92.71 0) (unit 1)
     (in_bom yes) (on_board yes) (fields_autoplaced)
-    (property "Reference" "#PWR045" (id 0) (at 125.73 99.06 0)
+    (property "Reference" "#PWR046" (id 0) (at 125.73 99.06 0)
       (effects (font (size 1.27 1.27)) hide)
     )
@@
       (effects (font (size 1.27 1.27)) (justify right))
     )
-    (property "Footprint" "Resistor_SMD:R_0402_1005Metric" (id 2) (at 85.09 111.76 0)
+    (property "Footprint" "4k7:RESC2013X65N" (id 2) (at 85.09 111.76 0)
       (effects (font (size 1.27 1.27)) (justify left) hide)
     )
@@
       (effects (font (size 1.27 1.27)) (justify right))
     )
-    (property "Footprint" "Resistor_SMD:R_0402_1005Metric" (id 2) (at 137.16 87.63 0)
+    (property "Footprint" "4k7:RESC2013X65N" (id 2) (at 137.16 87.63 0)
       (effects (font (size 1.27 1.27)) (justify left) hide)
     )
@@
   (symbol (lib_id "Connector:TestPoint") (at 114.3 97.155 0) (unit 1)
     (in_bom yes) (on_board yes) (fields_autoplaced)
-    (property "Reference" "TP11" (id 0) (at 116.84 92.5829 0)
+    (property "Reference" "TP12" (id 0) (at 116.84 92.5829 0)
       (effects (font (size 1.27 1.27)) (justify left))
     )
@@
       (effects (font (size 1.27 1.27)) (justify left))
     )
-    (property "Footprint" "TestPoint:TestPoint_Pad_D2.5mm" (id 2) (at 119.38 97.155 0)
-      (effects (font (size 1.27 1.27)) hide)
-    )
+    (property "Footprint" "TestPoint:TestPoint_Pad_D2.0mm" (id 2) (at 119.38 97.155 0)
+      (effects (font (size 1.27 1.27)) hide)
+    )
