File: PCB/main/sensing.kicad_sch (KiCad schematic)
At the start: 9 parts, among them J6 Conn_01x02_Male, J7 Conn_01x02_Male, J8 Conn_01x02_Male, J9 Conn_01x02_Male, U2 DS18B20Z, U3 ALS-PDIC15-21B/TR8

Commit message: Schematics v0.1.1 & PCB v0.01
Parts:
- U3: footprint OptoDevice:Vishay_MINICAST-3Pin -> ALS_Light:LED-SMD_1206-4P-L3.2-W1.5-TR
Changed lines of the file:
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@@
     (property "Reference" "U3" (id 0) (at 228.135 121.92 0))
     (property "Value" "ALS-PDIC15-21B/TR8" (id 1) (at 228.135 124.46 0))
-    (property "Footprint" "OptoDevice:Vishay_MINICAST-3Pin" (id 2) (at 228.6 142.875 0)
+    (property "Footprint" "ALS_Light:LED-SMD_1206-4P-L3.2-W1.5-TR" (id 2) (at 228.6 142.875 0)
       (effects (font (size 1.27 1.27)) hide)
     )
