File: PCB/main/sensing.kicad_sch (KiCad schematic)
At the start: 9 parts, among them J6 Conn_01x02_Male, J7 Conn_01x02_Male, J8 Conn_01x02_Male, J9 Conn_01x02_Male, U2 DS18B20Z, U3 ALS-PDIC15-21B/TR8

Commit message: v1.0 BOM, Gerbers & Final Designs
Parts:
- removed C8: 10uF, 10uF_0804:CAPC2012X145N, symbol pspice:C
- added C10: 10uF, 10uF_0804:CAPC2012X145N, symbol Device:C_Small
- added C7, C8, C9: 10nF, Capacitor_SMD:C_0402_1005Metric, symbol Device:C_Small
- J6: renamed from J7; JLC Part Number (none) -> C122410; LCSC (none) -> C122410; Price (none) -> 0.7097
- J7: renamed from J6; JLC Part Number (none) -> C122410; LCSC (none) -> C122410; Price (none) -> 0.7097
- J8, J9: JLC Part Number (none) -> C122410; LCSC (none) -> C122410; Price (none) -> 0.7097
- R17: renamed from R16; JLC Part Number (none) -> C21190; LCSC (none) -> C21190; Price (none) -> 0.0011
- R18: renamed from R17; JLC Part Number (none) -> C21190; LCSC (none) -> C21190; Price (none) -> 0.0011
- U2: JLC Part Number (none) -> C695837; LCSC (none) -> C695837; Price (none) -> 1.1052
- U3: JLC Part Number (none) -> C131243; LCSC (none) -> C131243; Price (none) -> 0.4279
Connections:
- net GND: now also C10.2, C7.1, C8.2, C9.2
- net at J9.2 (Pin_2), R18.1, U3.1 (OUT): now also C10.1
- net at J6.1 (Pin_1), U3.3 (Vs): now also C8.1
- net at J7.2 (Pin_2), R17.1, U2.3 (VDD): now also C7.2
- net at J8.2 (Pin_2), R17.2, U2.4 (DQ): now also C9.1
Other:
- title: (none) -> Sensing Submodule
- moved on the sheet: J6, J7, R18
