File: PCB/main/outputs.kicad_sch (KiCad schematic)
At the start: 0 parts

Commit message: Added sheet details to schematic
Other:
- company: (none) -> UCT
Changed lines of the file:
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@@
 (kicad_sch (version 20211123) (generator eeschema)
   (paper "A4")
+  (title_block
+    (date "2022-03-02")
+    (rev "v0.0")
+    (company "UCT")
+    (comment 2 "Group 7")
+    (comment 3 "@Checked By: ")
+    (comment 4 "@Authors: Ryan Jones, Alex Cargill & Devlin Trafford")
+  )
   (text "Not sure if you want this here:\n\nGP LEDS\nPushButton or 2 for testing\nUSB Connector\nTesting Connector\nJumpers for debugging and inserting signals"
     (at 126.365 86.36 0)
