File: PCB/main/main.kicad_pcb (KiCad board)
At the start: 2 copper layers, 4 parts, among them J1 Conn_01x33_Female, J2 Conn_01x33_Female, J3 Conn_01x33_Female, J4 Conn_01x33_Female

Commit message: Power Module v0.03
Other:
- board outline added: 88.9 x 53.3 mm
Changed lines of the file:
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@@
   )
   (gr_rect (start 173.99 91.44) (end 184.15 101.6) (layer "F.SilkS") (width 0.1) (fill none))
-  (gr_line (start 184.15 69.85) (end 184.15 123.19) (layer "F.Fab") (width 0.1))
-  (gr_line (start 95.25 123.19) (end 95.25 69.85) (layer "F.Fab") (width 0.1))
-  (gr_line (start 95.25 69.85) (end 184.15 69.85) (layer "F.Fab") (width 0.1))
-  (gr_line (start 184.15 123.19) (end 95.25 123.19) (layer "F.Fab") (width 0.1))
+  (gr_line (start 184.15 69.85) (end 184.15 123.19) (layer "Edge.Cuts") (width 0.1))
+  (gr_line (start 95.25 123.19) (end 95.25 69.85) (layer "Edge.Cuts") (width 0.1))
+  (gr_line (start 95.25 69.85) (end 184.15 69.85) (layer "Edge.Cuts") (width 0.1))
+  (gr_line (start 184.15 123.19) (end 95.25 123.19) (layer "Edge.Cuts") (width 0.1))
   (gr_rect (start 173.99 91.44) (end 184.15 101.6) (layer "F.Fab") (width 0.1) (fill none))
   (gr_text "USB" (at 179.07 96.52) (layer "F.SilkS")

Commit message: Schematics v0.1.1 & PCB v0.01
Parts:
- removed J1, J4: Conn_01x33_Female, Connector_PinHeader_2.54mm:PinHeader_1x33_P2.54mm_Vertical
- added BT1: 18650 Battery, bat_holder:KEYSTONE-1042, F.Cu at (137.0, 104.5)
- added C1: 1u, 1uF_0804:CAPC1608X90N, F.Cu at (148.9, 130.1)
- added C10: 100n, Capacitor_SMD:C_0402_1005Metric, F.Cu at (146.5, 87.8)
- added C11: 100n, Capacitor_SMD:C_0402_1005Metric, F.Cu at (146.5, 91.8)
- added C12: 22p, 22pF_0804:CAPC1608X90N, F.Cu at (153.8, 80.9)
- added C13: 22p, 22pF_0804:CAPC1608X90N, F.Cu at (162.2, 79.0)
- added C2: 10uF, 10uF_0804:CAPC2012X145N, F.Cu at (115.0, 120.8)
- added C3: 10uF, 10uF_0804:CAPC2012X145N, F.Cu at (99.2, 117.8)
- added C4: 1u, 1uF_0804:CAPC1608X90N, F.Cu at (97.6, 131.1)
- added C5: 1u, 1uF_0804:CAPC1608X90N, F.Cu at (115.0, 134.2)
- added C6: 1u, 1uF_0804:CAPC1608X90N, F.Cu at (117.5, 133.8)
- added C7: 1u, 1uF_0804:CAPC1608X90N, F.Cu at (107.0, 132.1)
- added C8: 10uF, 10uF_0804:CAPC2012X145N, F.Cu at (137.5, 77.2)
- added C9: 47n, 47nF_0804:CAPC1608X90N, F.Cu at (114.7, 127.3)
- added D1: 1N5819WS, Diode_SMD:D_SOD-323, F.Cu at (142.2, 137.9)
- added D2: 1N5819WS, Diode_SMD:D_SOD-323, F.Cu at (144.9, 137.4)
- added D3: Green LED, Green_LED:LEDC1608X50N, F.Cu at (110.4, 117.7)
- added D4: Red LED, Red_LED:LEDC1608X70N, F.Cu at (112.1, 121.6)
- added D5: 1N5819WS, Diode_SMD:D_SOD-323, F.Cu at (115.6, 131.7)
- added D6: LED, LED_SMD:LED_0805_2012Metric, F.Cu at (157.6, 95.3)
- added D7: LED, LED_SMD:LED_0805_2012Metric, F.Cu at (155.7, 71.2)
- added D8: LED, LED_SMD:LED_0805_2012Metric, F.Cu at (155.5, 90.8)
- added IC1: TP4056-42-ESOP8, TP4506:SOIC127P600X175-9N, F.Cu at (104.6, 119.7)
- added IC2: AMS1117-3.3, AMS1117-3.3V:SOT229P700X180-4N, F.Cu at (122.6, 135.2)
- added IC3: AT24C256C-SSHL-T, 3088_uC:SOIC127P600X175-8N, F.Cu at (142.7, 95.0)
- added J5: MICROXNJ, MICROXNJ:MICROXNJ, F.Cu at (135.9, 133.0)
- added J6: Conn_01x02_Male, conn_Molex_01_02_vert:53398-0271, F.Cu at (107.7, 74.3)
- added J7: Conn_01x02_Male, conn_Molex_01_02_vert:53398-0271, F.Cu at (116.8, 74.3)
- added J8: Conn_01x02_Male, conn_Molex_01_02_vert:53398-0271, F.Cu at (131.7, 74.4)
- added J9: Conn_01x02_Male, conn_Molex_01_02_vert:53398-0271, F.Cu at (140.4, 74.4)
- added Q1: AO3401A, AO3401A:SOT95P280X125-3N, F.Cu at (148.9, 132.9)
- added Q2: AO3401A, AO3401A:SOT95P280X125-3N, F.Cu at (100.4, 131.6)
- added Q3: AO3401A, AO3401A:SOT95P280X125-3N, F.Cu at (115.5, 137.4)
- added R1: 0R, 0R:RESC2013X65N, F.Cu at (118.0, 121.7)
- added R10: 0R, 0R:RESC2013X65N, F.Cu at (95.5, 129.4)
- added R11: 1k2, 1k:RESC1608X55N, F.Cu at (109.5, 121.0)
- added R12: 0R, 0R:RESC2013X65N, F.Cu at (112.5, 135.2)
- added R13: 3.3k, 3k3:RESC1608X55N, F.Cu at (118.5, 130.7)
- added R14: 4.7k, 4k7:RESC2013X65N, F.Cu at (118.4, 128.6)
- added R15: 0R, 0R:RESC2013X65N, F.Cu at (104.2, 132.8)
- added R16: 1k, 1k:RESC1608X55N, F.Cu at (107.1, 77.4)
- added R17: 1k, 1k:RESC1608X55N, F.Cu at (139.8, 77.2)
- added R18: 4.7k, 4k7:RESC2013X65N, F.Cu at (145.5, 89.8)
- added R19: 4.7k, 4k7:RESC2013X65N, F.Cu at (166.0, 80.6)
- added R2: 0R, 0R:RESC2013X65N, F.Cu at (142.2, 134.2)
- added R20: 1.5k, 4k7:RESC2013X65N, F.Cu at (152.5, 87.8)
- added R21: 1.5k, 4k7:RESC2013X65N, F.Cu at (182.2, 73.3)
- added R22: 1.5k, 4k7:RESC2013X65N, F.Cu at (150.5, 90.8)
- added R3: 0R, 0R:RESC2013X65N, F.Cu at (129.0, 137.8)
- added R4: 0R, 0R:RESC2013X65N, F.Cu at (139.2, 131.2)
- added R5: 100Ω, 100_ohm:RESC3116X65N, F.Cu at (155.9, 135.3)
- added R6: 4.7k, 4k7:RESC2013X65N, F.Cu at (148.7, 136.1)
- added R7: 4.7k, 4k7:RESC2013X65N, F.Cu at (148.7, 138.5)
- added R8: 1kΩ, 1k:RESC1608X55N, F.Cu at (104.9, 115.8)
- added R9: 1kΩ, 1k:RESC1608X55N, F.Cu at (99.4, 121.0)
- added TP1: TestPoint, TestPoint:TestPoint_Pad_D2.0mm, F.Cu at (144.9, 133.3)
- added TP10: TestPoint, TestPoint:TestPoint_Pad_D2.0mm, F.Cu at (161.0, 120.1)
- added TP11: TestPoint, TestPoint:TestPoint_Pad_D2.0mm, F.Cu at (164.7, 120.1)
- added TP12: TestPoint, TestPoint:TestPoint_Pad_D2.0mm, F.Cu at (122.8, 119.8)
- added TP13: TestPoint, TestPoint:TestPoint_Pad_D2.0mm, F.Cu at (123.5, 128.0)
- added TP2: TestPoint, TestPoint:TestPoint_Pad_D2.0mm, F.Cu at (152.1, 136.7)
- added TP3: TestPoint, TestPoint:TestPoint_Pad_D2.0mm, F.Cu at (128.9, 133.7)
- added TP4: TestPoint, TestPoint:TestPoint_Pad_D2.0mm, F.Cu at (142.6, 129.4)
- added TP5: TestPoint, TestPoint:TestPoint_Pad_D2.0mm, F.Cu at (153.2, 132.1)
- added TP6: TestPoint, TestPoint:TestPoint_Pad_D2.0mm, F.Cu at (104.2, 129.1)
- added TP7: TestPoint, TestPoint:TestPoint_Pad_D2.0mm, F.Cu at (109.7, 134.2)
- added TP8: TestPoint, TestPoint:TestPoint_Pad_D2.0mm, F.Cu at (179.0, 136.8)
- added TP9: TestPoint, TestPoint:TestPoint_Pad_D2.0mm, F.Cu at (133.3, 89.7)
- added U1: LM393, LMS393DRG:SOIC127P600X175-8N, F.Cu at (104.3, 136.8)
- added U2: DS18B20Z, Package_SO:SOIC-8_3.9x4.9mm_P1.27mm, F.Cu at (112.7, 78.1)
- added U3: ALS-PDIC15-21B/TR8, OptoDevice:Vishay_MINICAST-3Pin, F.Cu at (125.9, 75.8)
- added U4: CH340G, 3088_uC:SOIC127P600X180-16N, F.Cu at (173.1, 75.2)
- added Y1: YSX321SL, 3088_uC:YSX321SL, F.Cu at (158.4, 78.5)
- J2, J3: moved to B.Cu
- moved J2 7.96 mm to (179.4, 84.1), turned to 90 degrees
- moved J3 7.91 mm to (179.4, 124.7), turned to 90 degrees
Routing:
- net +5V: track 0.00 -> 48.6 mm
- net /Power/BAT +: track 0.00 -> 33.5 mm
- net Net-(C2-Pad1): track 0.00 -> 23.5 mm
- net Net-(C7-Pad1): track 0.00 -> 15.8 mm
- net Net-(C5-Pad1): track 0.00 -> 14.6 mm
- net Net-(D4-Pad1): track 0.00 -> 13.4 mm
- net +3V0: track 0.00 -> 12.8 mm
- net Net-(C1-Pad1): track 0.00 -> 11.3 mm, vias 0 -> 2
- net Net-(D1-Pad2): track 0.00 -> 8.73 mm
- net Net-(J5-Pad3): track 0.00 -> 7.35 mm
- net Net-(J5-Pad2): track 0.00 -> 7.21 mm
- net /Power/UVLO_OUT: track 0.00 -> 6.60 mm
- net /Power/BATOUT: track 0.00 -> 6.01 mm
- net Net-(Q1-Pad1): track 0.00 -> 5.76 mm
- net Net-(C4-Pad1): track 0.00 -> 4.86 mm
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- added copper zone on F.Cu, net GND
Other:
- board size 88.9 x 53.3 mm -> 100 x 70 mm
- board text removed: "USB"

Commit message: Schematics v0.1.1 & PCB v0.01
Parts:
- U3: footprint OptoDevice:Vishay_MINICAST-3Pin -> ALS_Light:LED-SMD_1206-4P-L3.2-W1.5-TR
- moved R21 58.1 mm to (149.4, 121.3)
- moved U4 53.3 mm to (142.3, 118.7), turned to 90 degrees
- moved TP9 50.9 mm to (176.9, 115.8)
- moved D7 47.0 mm to (149.5, 117.8), turned to 180 degrees
- moved C13 43.1 mm to (161.5, 122.1), turned to 180 degrees
- moved Y1 41.4 mm to (157.2, 119.9), turned to -90 degrees
- moved C12 39.2 mm to (160.8, 119.5), turned to 90 degrees
- moved R18 36.8 mm to (170.6, 116.8), turned to 90 degrees
- moved R19 36.8 mm to (172.9, 116.8)
- moved R22 36.6 mm to (125.7, 117.7), turned to 90 degrees
- moved R20 33.6 mm to (152.9, 121.3)
- moved IC3 32.7 mm to (165.6, 118.3)
- moved D8 32.5 mm to (135.8, 116.7), turned to 90 degrees
- moved C10 28.9 mm to (117.6, 87.3), turned to 180 degrees
- moved D6 22.4 mm to (152.5, 117.1), turned to 90 degrees
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Other:
- board text added: "+"
- board text added: "-"
- board text added: "EEE3088F Group 7 v0.01"

Commit message: Gerber, DRC text report, PCB v0.02
Parts:
- removed TP9: TestPoint, TestPoint:TestPoint_Pad_D2.0mm
- moved C10 62.5 mm to (179.8, 93.2), turned to 90 degrees
- moved C11 35.6 mm to (182.1, 93.3), turned to 90 degrees
- moved R22 24.3 mm to (149.7, 121.1), turned to 180 degrees
- moved TP11 14.7 mm to (185.9, 120.7)
- moved TP12 12.2 mm to (124.7, 128.5)
- moved TP10 11.3 mm to (185.8, 117.3)
- moved R18 9.55 mm to (179.9, 118.7)
- moved TP13 9.53 mm to (128.2, 128.4)
- moved IC3 5.78 mm to (171.3, 119.3)
- moved R21 5.06 mm to (149.8, 116.3)
- moved D7 4.93 mm to (154.2, 116.3), turned to 0 degrees
- moved C13 4.63 mm to (164.0, 118.2)
- moved R19 4.28 mm to (177.0, 117.9)
- moved R20 4.12 mm to (149.8, 118.7)
- moved C12 3.29 mm to (164.0, 120.4), turned to 180 degrees
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Routing:
- net +3V0: track 12.8 -> 210.6 mm, vias 0 -> 2
- net /PA3: track 0.00 -> 68.6 mm
- net /PA9: track 0.00 -> 57.4 mm
- net GND: track 1.14 -> 54.3 mm, vias 0 -> 13
- net /Power/VPolarity: track 3.07 -> 44.7 mm, vias 0 -> 2
- net /PA10: track 0.00 -> 37.3 mm
- net Net-(J8-Pad2): track 0.00 -> 35.6 mm
- net /PB6: track 0.00 -> 28.1 mm
- net /PB7: track 0.00 -> 25.2 mm
- net Net-(C8-Pad1): track 0.00 -> 24.5 mm
- net /Power/USB (D+): track 4.45 -> 23.9 mm
- net Net-(U4-Pad7): track 0.00 -> 17.7 mm
- net Net-(U4-Pad8): track 0.00 -> 15.9 mm
- net /PA2: track 0.00 -> 15.3 mm, vias 0 -> 1
- net /PA1: track 0.00 -> 9.57 mm
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- added copper zone on B.Cu, net GND
Other:
- outline, holes or cut-outs redrawn
- board text added: "EEE3088F Group 7 v0.02"
- board text removed: "EEE3088F Group 7 v0.01"

Commit message: Upload Week 6 Handin
Parts:
- added G***: LOGO, 3088_aux_fps:qr_code, F.Cu at (101.8, 89.9)
Routing:
- net /PA2: vias 1 -> 2
- net GND: vias 13 -> 12

Commit message: v1.0 BOM, Gerbers & Final Designs
Parts:
- removed Q3: AO3401A, AO3401A:SOT95P280X125-3N
- removed TP12, TP13: TestPoint, TestPoint:TestPoint_Pad_D2.0mm
- added C14: 22p, 22pF_0804:CAPC1608X90N, F.Cu at (164.4, 131.0)
- added C15: 22p, 22pF_0804:CAPC1608X90N, F.Cu at (157.5, 132.0)
- added D9: LED, LED_SMD:LED_0805_2012Metric, F.Cu at (145.8, 119.3)
- added G***: LOGO, 3088_aux_fps:github, F.Cu at (101.6, 76.2)
- added IC4: TXS0108EPWR, 3088_uC:SOP65P640X120-20N, F.Cu at (137.2, 131.1)
- added J10: Conn_01x02_Male, conn_Molex_01_02_vert:53398-0271, F.Cu at (124.6, 90.5)
- added J11: Conn_01x02_Male, conn_Molex_01_02_vert:53398-0271, F.Cu at (164.8, 121.1)
- added J12: Conn_01x02_Male, conn_Molex_01_02_vert:53398-0271, F.Cu at (135.8, 121.4)
- added J13: Conn_01x02_Male, conn_Molex_01_02_vert:53398-0271, F.Cu at (124.2, 119.3)
- added R23: 1.5k, 4k7:RESC2013X65N, F.Cu at (142.1, 119.3)
- added TP9: TestPoint, TestPoint:TestPoint_Pad_D2.0mm, F.Cu at (183.1, 84.1)
- C1, C4: value 1u -> 10uF; footprint 1uF_0804:CAPC1608X90N -> 10uF_0804:CAPC2012X145N
- C10: value 100n -> 10uF; footprint Capacitor_SMD:C_0402_1005Metric -> 10uF_0804:CAPC2012X145N
- C11: value 100n -> 47n; footprint Capacitor_SMD:C_0402_1005Metric -> 47nF_0804:CAPC1608X90N
- C12, C13: value 22p -> 100n; footprint 22pF_0804:CAPC1608X90N -> Capacitor_SMD:C_0402_1005Metric
- C7: value 1u -> 10nF; footprint 1uF_0804:CAPC1608X90N -> Capacitor_SMD:C_0402_1005Metric
- C8: value 10uF -> 10nF; footprint 10uF_0804:CAPC2012X145N -> Capacitor_SMD:C_0402_1005Metric
- C9: value 47n -> 10nF; footprint 47nF_0804:CAPC1608X90N -> Capacitor_SMD:C_0402_1005Metric
- D1: value 1N5819WS -> Red LED; footprint Diode_SMD:D_SOD-323 -> Red_LED:LEDC1608X70N
- D3: value Green LED -> 1N5819WS; footprint Green_LED:LEDC1608X50N -> Diode_SMD:D_SOD-323
- D4: value Red LED -> 1N5819WS; footprint Red_LED:LEDC1608X70N -> Diode_SMD:D_SOD-323
- D5: value 1N5819WS -> Green LED; footprint Diode_SMD:D_SOD-323 -> Green_LED:LEDC1608X50N
- D6: value LED -> Red LED; footprint LED_SMD:LED_0805_2012Metric -> Red_LED:LEDC1608X70N
- IC2: value AMS1117-3.3 -> LM393DR2G; footprint AMS1117-3.3V:SOT229P700X180-4N -> LMS393DRG:SOIC127P600X175-8N
- J5: footprint MICROXNJ:MICROXNJ -> 3088_power:MICROXNJ
- Q1: value AO3401A -> MMBT3904; footprint AO3401A:SOT95P280X125-3N -> Package_TO_SOT_SMD:SOT-23
- R11: value 1k2 -> 0R; footprint 1k:RESC1608X55N -> 0R:RESC2013X65N
- R13: value 3.3k -> 1k2; footprint 3k3:RESC1608X55N -> 1k:RESC1608X55N
- R14, R18: value 4.7k -> 1k; footprint 4k7:RESC2013X65N -> 1k:RESC1608X55N
- R15: value 0R -> 10k; footprint 0R:RESC2013X65N -> 10k:RESC1005X40N
- R16: value 1k -> 0R; footprint 1k:RESC1608X55N -> 0R:RESC2013X65N
- R20: value 1.5k -> 4.7k
- R5: value 100Ω -> 0R; footprint 100_ohm:RESC3116X65N -> 0R:RESC2013X65N
- R8, R9: value 1kΩ -> 1k
- U1: value LM393 -> HT75xx-1-SOT89; footprint LMS393DRG:SOIC127P600X175-8N -> Package_TO_SOT_SMD:SOT-89-3
- moved TP5 71.4 mm to (94.0, 92.2)
- moved C7 59.3 mm to (128.4, 76.8)
- moved R18 56.6 mm to (143.0, 75.8), turned to 180 degrees
- moved C12 55.8 mm to (131.3, 75.2)
- moved Q1 55.7 mm to (93.3, 131.3), turned to 90 degrees
- moved C9 55.4 mm to (137.5, 76.8), turned to -90 degrees
- moved R16 53.1 mm to (106.0, 130.5)
- moved J6 48.6 mm to (156.4, 74.3)
- moved IC3 48.0 mm to (133.3, 89.9), turned to 90 degrees
- moved R2 47.6 mm to (94.7, 138.2), turned to 180 degrees
- moved C13 46.2 mm to (129.8, 87.1), turned to 90 degrees
- moved R6 45.3 mm to (103.3, 135.9), turned to 180 degrees
- moved TP10 45.3 mm to (143.2, 132.7)
- moved R7 41.6 mm to (107.1, 135.9)
- moved C10 39.9 mm to (143.0, 77.8), turned to 180 degrees
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Connections:
- C10 pad 1: GND -> Net-(C10-Pad1)
- C10 pad 2: +3V0 -> GND
- C11 pad 2: +3V0 -> +3V3
- C12 pad 2: Net-(C12-Pad2) -> +3V3
- C13 pad 2: Net-(C13-Pad2) -> +3V3
- C3 pad 1: /Power/BAT + -> Net-(C3-Pad1)
- C4 pad 1: Net-(C4-Pad1) -> /Power/BAT +
- C6 pad 1: +3V0 -> Net-(C6-Pad1)
- C7 pad 1: Net-(C7-Pad1) -> GND
- C7 pad 2: GND -> Net-(C7-Pad2)
- C9 pad 1: GND -> Net-(C9-Pad1)
- C9 pad 2: +3V0 -> GND
- D1 pad 1: +5V -> GND
- D1 pad 2: Net-(D1-Pad2) -> /Power/USBDETECT
- D2 pad 1: Net-(D2-Pad1) -> Net-(C2-Pad1)
- D2 pad 2: Net-(D1-Pad2) -> Net-(C3-Pad1)
- D3 pad 1: Net-(D3-Pad1) -> +5V
- D3 pad 2: Net-(C2-Pad1) -> Net-(D3-Pad2)
- D4 pad 2: Net-(C2-Pad1) -> Net-(D3-Pad2)
- D5 pad 1: Net-(C5-Pad1) -> Net-(D5-Pad1)
- D5 pad 2: +3V0 -> Net-(C1-Pad1)
- D6 pad 2: +3V0 -> Net-(C1-Pad1)
- D7 pad 2: +3V0 -> +3V3
- D8 pad 1: /PA9 -> Net-(D8-Pad1)
- D8 pad 2: +3V0 -> +3V3
- IC1 pad 4: Net-(C2-Pad1) -> Net-(C1-Pad1)
- IC1 pad 8: Net-(C2-Pad1) -> Net-(C1-Pad1)
- IC2 pad 2: +3V0 -> Net-(IC2-Pad2)
- IC2 pad 3: Net-(C5-Pad1) -> Net-(C6-Pad1)
- IC2 pad 4: unconnected-(IC2-Pad4) -> GND
- IC3 pad 5: /PB7 -> Net-(IC3-Pad5)
- IC3 pad 6: /PB6 -> Net-(IC3-Pad6)
- IC3 pad 8: +3V0 -> +3V3
- J5 pad 1: Net-(D1-Pad2) -> Net-(D3-Pad2)
- J5 pad MH1: GND -> (no net)
- J5 pad MH2: GND -> (no net)
- J5 pad MH3: GND -> (no net)
- J5 pad MH4: GND -> (no net)
- J5 pad MP1: GND -> (no net)
- J5 pad MP2: GND -> (no net)
- J6 pad 1: +3V0 -> Net-(C8-Pad1)
- J6 pad 2: Net-(J6-Pad2) -> +3V3
- J7 pad 1: Net-(J7-Pad1) -> +3V3
- J7 pad 2: +3V0 -> Net-(C7-Pad2)
- J8 pad 2: Net-(J8-Pad2) -> Net-(C9-Pad1)
- J9 pad 2: Net-(C8-Pad1) -> Net-(C10-Pad1)
- Q1 pad 1: Net-(Q1-Pad1) -> Net-(IC2-Pad1)
- Q1 pad 2: /Power/VPolarity -> Net-(Q1-Pad2)
- Q1 pad 3: Net-(C1-Pad1) -> /Power/BATOUT
- Q2 pad 2: /Power/BATOUT -> Net-(Q2-Pad2)
- Q2 pad 3: Net-(C4-Pad1) -> Net-(C5-Pad1)
- R1 pad 1: Net-(C2-Pad1) -> Net-(C1-Pad1)
- R1 pad 2: /Power/VPolarity -> +5V
- R10 pad 1: Net-(C4-Pad1) -> /Power/UVLO_OUT
- R10 pad 2: /Power/BAT + -> Net-(Q1-Pad2)
- R11 pad 1: Net-(IC1-Pad2) -> Net-(C5-Pad1)
- R11 pad 2: GND -> /Power/BAT +
- R12 pad 1: Net-(C5-Pad1) -> /Power/BATOUT
- R12 pad 2: /Power/UVLO_OUT -> Net-(Q2-Pad2)
- R13 pad 1: Net-(IC2-Pad1) -> Net-(IC1-Pad2)
- R13 pad 2: +3V0 -> GND
- R14 pad 1: GND -> +3V0
- R14 pad 2: Net-(IC2-Pad1) -> Net-(IC2-Pad2)
- R15 pad 1: Net-(C7-Pad1) -> Net-(IC2-Pad2)
- R15 pad 2: /Power/BATOUT -> GND
- R16 pad 1: Net-(J6-Pad2) -> Net-(C6-Pad1)
- R16 pad 2: Net-(J8-Pad2) -> /Power/BATOUT
- R17 pad 1: Net-(C8-Pad1) -> Net-(C7-Pad2)
- R17 pad 2: GND -> Net-(C9-Pad1)
- R18 pad 1: /PB7 -> Net-(C10-Pad1)
- R18 pad 2: +3V0 -> GND
- R19 pad 1: /PB6 -> /PB7
- R19 pad 2: +3V0 -> +3V3
- R2 pad 1: Net-(C1-Pad1) -> Net-(C2-Pad1)
- R2 pad 2: +5V -> /Power/UVLO_OUT
- R20 pad 1: /PA9 -> /PB6
- R20 pad 2: Net-(D6-Pad1) -> +3V3
- R21 pad 1: /PA10 -> /PA9
- R22 pad 1: GND -> /PA10
- R22 pad 2: /PA9 -> Net-(D8-Pad1)
- R3 pad 1: /Power/USB (D+) -> +3V0
- R3 pad 2: Net-(J5-Pad3) -> Net-(C3-Pad1)
- R4 pad 1: /Power/USB (D-) -> /Power/USB (D+)
- R4 pad 2: Net-(J5-Pad2) -> Net-(J5-Pad3)
- R5 pad 1: Net-(Q1-Pad1) -> /Power/USB (D-)
- R5 pad 2: GND -> Net-(J5-Pad2)
- R6 pad 1: Net-(D2-Pad1) -> Net-(D4-Pad1)
- R7 pad 2: Net-(D2-Pad1) -> Net-(D4-Pad1)
- R8 pad 1: Net-(D3-Pad1) -> Net-(D5-Pad1)
- R9 pad 1: Net-(D4-Pad1) -> Net-(D6-Pad1)
- TP10 pad 1: /PB6 -> Net-(IC4-Pad3)
- TP11 pad 1: /PB7 -> Net-(IC4-Pad4)
- TP5 pad 1: /Power/VPolarity -> /Power/BAT +
- U1 pad 2: /Power/VRegulated -> Net-(C2-Pad1)
- U1 pad 3: Net-(C7-Pad1) -> Net-(C3-Pad1)
- U2 pad 3: Net-(J6-Pad2) -> Net-(C7-Pad2)
- U2 pad 4: Net-(J8-Pad2) -> Net-(C9-Pad1)
- U3 pad 1: Net-(C8-Pad1) -> Net-(C10-Pad1)
- U3 pad 3: Net-(J7-Pad1) -> Net-(C8-Pad1)
- U4 pad 16: +3V0 -> +3V3
- U4 pad 2: /PA10 -> Net-(J13-Pad1)
- U4 pad 3: /PA9 -> Net-(J12-Pad1)
- U4 pad 4: +3V0 -> +3V3
- U4 pad 5: /Power/USB (D+) -> Net-(IC4-Pad3)
- U4 pad 6: /Power/USB (D-) -> Net-(IC4-Pad4)
- Y1 pad 2: Net-(C13-Pad2) -> Net-(C15-Pad2)
- Y1 pad 4: Net-(C12-Pad2) -> Net-(C14-Pad2)
Routing:
- net +3V3: track 0.00 -> 128.6 mm, vias 0 -> 12
- net +3V0: track 210.6 -> 127.4 mm, vias 2 -> 6
- net /PA3: track 68.6 -> 5.05 mm
- net Net-(IC3-Pad5): track 0.00 -> 52.7 mm
- net /Power/VPolarity: track 44.7 -> 0.00 mm, vias 2 -> 0
- net GND: track 54.3 -> 14.7 mm, vias 12 -> 17
- net Net-(J8-Pad2): track 35.6 -> 0.00 mm
- net /PA9: track 57.4 -> 24.1 mm, vias 0 -> 2
- net /PA10: track 37.3 -> 5.27 mm
- net Net-(J13-Pad1): track 0.00 -> 30.0 mm, vias 0 -> 2
- net +5V: track 48.6 -> 78.3 mm
- net /PB6: track 28.1 -> 55.1 mm, vias 0 -> 2
- net Net-(C1-Pad1): track 11.3 -> 36.3 mm
- net Net-(D3-Pad2): track 0.00 -> 21.0 mm
- net Net-(J12-Pad1): track 0.00 -> 19.1 mm, vias 0 -> 2
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Other:
- board size 100 x 70 mm -> 96 x 70 mm
- board text added: "+3V"
- board text added: "+5V"
- board text added: "CHARGE"
- board text added: "EEE3088F Group 7 v1.0"
- board text added: "GitHub Link"
- board text added: "Ryan Jones Alex Cargill Devlin Trafford"
- board text added: "STDBY"
- board text added: "USB"
- board text added: "USB DETECT"
- board text removed: "EEE3088F Group 7 v0.02"
