File: PCB/main/power.kicad_sch (KiCad schematic)
At the start: 42 parts, among them IC1 TP4056-42-ESOP8, IC2 AMS1117-3.3, J5 MICROXNJ, Q1 AO3401A, Q2 AO3401A, Q3 AO3401A, U1 LM393

Commit message: Schematics v0.1.1 & PCB v0.01
Parts:
- added TP8: TestPoint, TestPoint:TestPoint_Pad_D2.0mm, symbol Connector:TestPoint
- BT1: footprint Battery:BatteryHolder_Keystone_1042_1x18650 -> bat_holder:KEYSTONE-1042
- D5: footprint Diode_THT:D_DO-41_SOD81_P10.16mm_Horizontal -> Diode_SMD:D_SOD-323
Connections:
- net GND: now also TP8.1
Changed lines of the file:
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@@
+    (stroke (width 0) (type default) (color 0 0 0 0))
+  )
+  (wire (pts (xy 33.02 110.49) (xy 33.02 116.84))
     (stroke (width 0) (type default) (color 0 0 0 0))
   )
@@
     (pin "2")
   )
+  (symbol (lib_id "power:GND") (at 33.02 116.84 0) (unit 1)
+    (in_bom yes) (on_board yes) (fields_autoplaced)
+    (property "Reference" "#PWR040" (id 0) (at 33.02 123.19 0)
+      (effects (font (size 1.27 1.27)) hide)
+    )
+    (property "Value" "GND" (id 1) (at 33.02 121.2834 0))
+    (property "Footprint" "" (id 2) (at 33.02 116.84 0)
+      (effects (font (size 1.27 1.27)) hide)
+    )
+    (property "Datasheet" "" (id 3) (at 33.02 116.84 0)
+      (effects (font (size 1.27 1.27)) hide)
+    )
+    (pin "1")
+  )
   (symbol (lib_id "power:GND") (at 257.81 53.34 0) (unit 1)
     (in_bom yes) (on_board yes) (fields_autoplaced)
@@
     (pin "2")
   )
+  (symbol (lib_id "Connector:TestPoint") (at 33.02 110.49 0) (unit 1)
+    (in_bom yes) (on_board yes) (fields_autoplaced)
+    (property "Reference" "TP8" (id 0) (at 34.417 106.3533 0)
+      (effects (font (size 1.27 1.27)) (justify left))
+    )
+    (property "Value" "TestPoint" (id 1) (at 34.417 108.8902 0)
+      (effects (font (size 1.27 1.27)) (justify left))
+    )
+    (property "Footprint" "TestPoint:TestPoint_Pad_D2.0mm" (id 2) (at 38.1 110.49 0)
+      (effects (font (size 1.27 1.27)) hide)
+    )
+    (property "Datasheet" "~" (id 3) (at 38.1 110.49 0)
+      (effects (font (size 1.27 1.27)) hide)
+    )
+    (pin "1")
+  )
   (symbol (lib_id "Device:LED") (at 186.69 34.29 90) (unit 1)
     (in_bom yes) (on_board yes)
@@
       (effects (font (size 1.27 1.27)) (justify left))
     )
-    (property "Footprint" "Diode_THT:D_DO-41_SOD81_P10.16mm_Horizontal" (id 2) (at 124.46 48.895 0)
+    (property "Footprint" "Diode_SMD:D_SOD-323" (id 2) (at 124.46 48.895 0)
       (effects (font (size 1.27 1.27)) hide)
     )
@@
       (effects (font (size 1.27 1.27)) (justify left))
     )
-    (property "Footprint" "Battery:BatteryHolder_Keystone_1042_1x18650" (id 2) (at 267.97 44.196 90)
-      (effects (font (size 1.27 1.27)) hide)
-    )
+    (property "Footprint" "bat_holder:KEYSTONE-1042" (id 2) (at 267.97 44.196 90)
+      (effects (font (size 1.27 1.27)) hide)
+    )

Commit message: v1.0 BOM, Gerbers & Final Designs
Parts:
- removed C1, C5, C7: 1u, 1uF_0804:CAPC1608X90N, symbol Device:C_Small
- removed IC2: AMS1117-3.3, AMS1117-3.3V:SOT229P700X180-4N, symbol AMS1117-3.3V:AMS1117-3.3
- removed Q1, Q3: AO3401A, AO3401A:SOT95P280X125-3N, symbol Transistor_FET:AO3401A
- removed R13: 3.3k, 3k3:RESC1608X55N, symbol Device:R_Small_US
- removed R5: 100Ω, 100_ohm:RESC3116X65N, symbol Device:R_Small_US
- removed U1: LM393, LMS393DRG:SOIC127P600X175-8N, symbol Comparator:LM393
- added C2, C3: 10uF, 10uF_0804:CAPC2012X145N, symbol Device:C_Small
- added IC2: LM393DR2G, LMS393DRG:SOIC127P600X175-8N, symbol LM393DR2G:LM393DR2G
- added Q1: MMBT3904, Package_TO_SOT_SMD:SOT-23, symbol Transistor_BJT:MMBT3904
- added R10, R16, R3: 0R, 0R:RESC2013X65N, symbol Device:R_Small_US
- added TP9: TestPoint, TestPoint:TestPoint_Pad_D2.0mm, symbol Connector:TestPoint
- added U1: HT75xx-1-SOT89, Package_TO_SOT_SMD:SOT-89-3, symbol Regulator_Linear:HT75xx-1-SOT89
- C1: renamed from C2; LCSC (none) -> C19702; Price $0.068 -> 0.068
- C4: renamed from C3; LCSC (none) -> C19702; Price $0.068 -> 0.068
- C5: renamed from C4; LCSC (none) -> C52923; Price $0.0037 -> 0.0037
- C6: LCSC (none) -> C52923; Price $0.0037 -> 0.0037
- D2: renamed from D5; LCSC (none) -> C191023
- D3: renamed from D1; LCSC (none) -> C191023
- D4: renamed from D2; LCSC (none) -> C191023
- D5: renamed from D3; LCSC (none) -> C72043; Price $0.0312 -> 0.0312
- D6: renamed from D4; LCSC (none) -> C84256; Price $0.0139 -> 0.0139
- IC1: LCSC (none) -> C16581; Price $0.2578 -> 0.2578
- J5: footprint MICROXNJ:MICROXNJ -> 3088_power:SHOUHAN_MICROXNJ; LCSC (none) -> C404969; Price $0.6496 -> 0.6496
- Q2: LCSC (none) -> C15127; Price $0.1774 -> 0.1774
- R1, R12, R2: LCSC (none) -> C17477
- R11: renamed from R10; LCSC (none) -> C17477
- R13: renamed from R11; LCSC (none) -> C22765; Price $0.0014 -> 0.0014
- R14: value 4.7k -> 1k; footprint 4k7:RESC2013X65N -> 1k:RESC1608X55N; Field5 (none) -> $0.0007; JLC Part Number C17673 -> C21190; LCSC (none) -> C21190; Price 0.0027 -> 0.0011
- R15: value 0R -> 10k; footprint 0R:RESC2013X65N -> 10k:RESC1005X40N; Field5 (none) -> $0.0007; JLC Part Number C17477 -> C25905; LCSC (none) -> C25905; Price 0.0024 -> 0.0007
- R4: renamed from R3; LCSC (none) -> C17477
- R5: renamed from R4; LCSC (none) -> C17477
- R6, R7: LCSC (none) -> C17673
- R8, R9: value 1kΩ -> 1k; JLC Part Number C25905 -> C21190; LCSC (none) -> C21190; Price $0.0007 -> 0.0011
Connections:
- net +3V3: now also R14.1, R3.1, TP9.1; no longer C6.1, D2.2 (A)
- net BAT +: now also TP5.1
- net BATOUT: now also R12.1, IC2.8 (VCC), Q1.3 (C), R16.2; no longer Q2.2 (S), R15.2
- net GND: now also R15.2, C2.2, C3.2, IC2.4 (GND), U1.1 (GND); no longer R14.1
- net UVLO_OUT: now also R2.2, R10.1; no longer R12.2
- net VCCBus: now also R1.2; no longer R2.2
- net at R14.2: now also R15.1, IC2.2 (INPUTSA_1)
- net at D2.1 (K): now also R2.1, C2.1, U1.2 (VIN); no longer R12.1
- removed net VPolarity: R1.2, TP5.1
- new net: C6.1, IC2.3 (INPUTSA_2), R16.1
- new net: C3.1, D2.2 (A), R3.2, U1.3 (VOUT)
- new net: Q1.2 (E), R10.2
- new net: Q2.2 (S), R12.2
- new net: IC2.1 (OUTPUTA), Q1.1 (B)
- no-connect marks 2 -> 5
Other:
- note added: "Test Points"
- note removed: "Input Polarity Protection Circuit"
- moved on the sheet: D2
